File: MiDi_Controller_Rev_2/MiDi_Controller_Rev_2.kicad_pcb (KiCad board)
At the start: 2 copper layers, 272.9 x 150 mm, 167 parts, among them J1 USB_C_Receptacle_USB2.0_16P, J10 Conn_01x24_Pin, J2 USB_C_Receptacle_USB2.0_16P, J3 DIN-5, J4 DIN-5, J5 Conn_01x03_Pin, J6 Display, J8 KEYPAD_LEDS, Q1 BC817, Q11 NMOS, Q12 NMOS, Q13 NMOS, Q17 NMOS, Q18 NMOS, Q19 NMOS, Q2 BC817, Q3 NMOS, Q5 NMOS, Q6 NMOS, Q7 NMOS, SW1 TS-1088-AR02016, SW11 SW_Push, SW13 SW_Push, SW15 SW_Push, SW16 SW_Push, SW17 SW_Push, SW2 TS-1088-AR02016, SW21 RotaryEncoder_Switch, SW23 SW_Push, SW24 SW_Push, SW25 SW_Push, SW29 SW_Push, SW3 SW_Push, SW30 SW_Push, SW31 SW_Push, SW35 RotaryEncoder_Switch, SW38 SW_Push, SW5 SW_Push, SW7 SW_Push, SW9 SW_Push, U1 CH340C, U2 ESP32-S3-WROOM-1, U3 H11L1, U4 AMS1117-3.3, U5 AMS1117-3.3, U7 MCP23017x-x-SO, U9 MCP23017x-x-SO

Commit message: Changed README.md so rev 1 lists actual problems, not a wide expression.
Parts:
- J10: footprint Connector_PinSocket_2.54mm:PinSocket_1x24_P2.54mm_Vertical -> Connector_PinHeader_2.54mm:PinHeader_1x24_P2.54mm_Horizontal
Routing:
- net VCC: track 235.7 -> 234.7 mm
